Commit message: Sync Arctos ROS 2 workspace updates

File: ros2/arctos_moveit_config/config/arctos_urdf.ros2_control.xacro (robot description, xacro)
@@ -75,18 +75,4 @@
                 <state_interface name="velocity"/>
             </joint>
-            <joint name="jaw1">
-                <command_interface name="position"/>
-                <state_interface name="position">
-                    <param name="initial_value">${initial_positions['jaw1']}</param>
-                </state_interface>
-                <state_interface name="velocity"/>
-            </joint>
-            <joint name="jaw2">
-                <command_interface name="position"/>
-                <state_interface name="position">
-                    <param name="initial_value">${initial_positions['jaw2']}</param>
-                </state_interface>
-                <state_interface name="velocity"/>
-            </joint>
         </ros2_control>
     </xacro:macro>

File: ros2/arctos_urdf_description/urdf/arctos.urdf (robot description, URDF)
Before this commit: robot arctos_urdf, 10 links, 9 joints
Links:
- removed link Gripper_1
- removed link Left_jaw_1
- removed link Right_jaw_1
- added link C_Core_Suction, mass 0.5810486809925093; collision mesh filename=package://arctos_urdf_description/meshes/C Core Suction.stl scale=0.001 0.001 0.001; visual mesh filename=package://arctos_urdf_description/meshes/C Core Suction.stl scale=0.001 0.001 0.001
Joints:
- removed joint gripper
- removed joint jaw1
- removed joint jaw2
- added joint suction_tool: type fixed, parent Link_6_1, child C_Core_Suction, origin xyz=0.0 -0.006085 0.0 rpy=0 0 0
- joint joint5: limit (none) -> lower=-1.57079632679 upper=1.57079632679 effort=100 velocity=2.0; type continuous -> revolute
- joint joint6: limit (none) -> lower=-3.14159265359 upper=3.14159265359 effort=100 velocity=2.0; type continuous -> revolute

File: ros2/arctos_urdf_description/urdf/arctos_urdf.xacro (robot description, xacro)
@@ -124,5 +124,5 @@
   </collision>
 </link>
-<link name="Gripper_1">
+<link name="C_Core_Suction">
   <inertial>
     <origin xyz="0.0036112727264542635 -0.014760653808445767 -0.00103677815369696" rpy="0 0 0"/>
@@ -131,14 +131,14 @@
   </inertial>
   <visual>
-    <origin xyz="-0.000193 0.319847 -0.570316" rpy="0 0 0"/>
-    <geometry>
-      <mesh filename="package://arctos_urdf_description/meshes/Gripper_1.stl" scale="0.001 0.001 0.001"/>
-    </geometry>
-    <material name="paint_metallic_blue_2"/>
-  </visual>
-  <collision>
-    <origin xyz="-0.000193 0.319847 -0.570316" rpy="0 0 0"/>
-    <geometry>
-      <mesh filename="package://arctos_urdf_description/meshes/Gripper_1.stl" scale="0.001 0.001 0.001"/>
+    <origin xyz="-0.000429 -0.008602 -0.624470" rpy="0 0 0"/>
+    <geometry>
+      <mesh filename="package://arctos_urdf_description/meshes/C Core Suction.stl" scale="0.001 0.001 0.001"/>
+    </geometry>
+    <material name="paint_metallic_blue_2"/>
+  </visual>
+  <collision>
+    <origin xyz="-0.000429 -0.008602 -0.624470" rpy="0 0 0"/>
+    <geometry>
+      <mesh filename="package://arctos_urdf_description/meshes/C Core Suction.stl" scale="0.001 0.001 0.001"/>
     </geometry>
   </collision>
@@ -161,44 +161,4 @@
     <geometry>
       <mesh filename="package://arctos_urdf_description/meshes/Link_6_1.stl" scale="0.001 0.001 0.001"/>
-    </geometry>
-  </collision>
-</link>
-<link name="Left_jaw_1">
-  <inertial>
-    <origin xyz="-0.011142702480351952 -0.009692440309284511 -0.009385792627785827" rpy="0 0 0"/>
-    <mass value="0.07369602565859415"/>
-    <inertia ixx="1.1e-05" iyy="6e-06" izz="1.4e-05" ixy="2e-06" iyz="-0.0" ixz="-0.0"/>
-  </inertial>
-  <visual>
-    <origin xyz="-0.007934 0.359845 -0.599867" rpy="0 0 0"/>
-    <geometry>
-      <mesh filename="package://arctos_urdf_description/meshes/Left_jaw_1.stl" scale="0.001 0.001 0.001"/>
-    </geometry>
-    <material name="paint_metallic_blue_2"/>
-  </visual>
-  <collision>
-    <origin xyz="-0.007934 0.359845 -0.599867" rpy="0 0 0"/>
-    <geometry>
-      <mesh filename="package://arctos_urdf_description/meshes/Left_jaw_1.stl" scale="0.001 0.001 0.001"/>
-    </geometry>
-  </collision>
-</link>
-<link name="Right_jaw_1">
-  <inertial>
-    <origin xyz="-0.008289104952972526 -0.009768535307719373 0.009395511902715814" rpy="0 0 0"/>
-    <mass value="0.07312902168719511"/>
-    <inertia ixx="1.1e-05" iyy="6e-06" izz="1.4e-05" ixy="-1e-06" iyz="0.0" ixz="-1e-06"/>
-  </inertial>
-  <visual>
-    <origin xyz="-0.007934 0.359845 -0.539867" rpy="0 0 0"/>
-    <geometry>
-      <mesh filename="package://arctos_urdf_description/meshes/Right_jaw_1.stl" scale="0.001 0.001 0.001"/>
-    </geometry>
-    <material name="paint_metallic_blue_2"/>
-  </visual>
-  <collision>
-    <origin xyz="-0.007934 0.359845 -0.539867" rpy="0 0 0"/>
-    <geometry>
-      <mesh filename="package://arctos_urdf_description/meshes/Right_jaw_1.stl" scale="0.001 0.001 0.001"/>
     </geometry>
   </collision>
@@ -228,34 +188,22 @@
   <axis xyz="-0.0 1.0 -0.0"/>
 </joint>
-<joint name="joint5" type="continuous">
+<joint name="joint5" type="revolute">
   <origin xyz="-0.039012 -0.121187 -0.001774" rpy="0 0 0"/>
   <parent link="Link_4_1"/>
   <child link="Link_5_1"/>
   <axis xyz="-1.0 -0.0 0.0"/>
-</joint>
-<joint name="gripper" type="fixed">
+  <limit lower="-1.57079632679" upper="1.57079632679" effort="100" velocity="2.0"/>
+</joint>
+<joint name="suction_tool" type="fixed">
   <origin xyz="0.0 -0.006085 0.0" rpy="0 0 0"/>
   <parent link="Link_6_1"/>
-  <child link="Gripper_1"/>
-</joint>
-<joint name="joint6" type="continuous">
+  <child link="C_Core_Suction"/>
+</joint>
+<joint name="joint6" type="revolute">
   <origin xyz="0.039204 -0.033835 0.0" rpy="0 0 0"/>
   <parent link="Link_5_1"/>
   <child link="Link_6_1"/>
   <axis xyz="-0.0 1.0 -0.0"/>
-</joint>
-<joint name="jaw1" type="prismatic">
-  <origin xyz="0.007741 -0.039998 0.029551" rpy="0 0 0"/>
-  <parent link="Gripper_1"/>
-  <child link="Left_jaw_1"/>
-  <axis xyz="-0.0 0.0 -1.0"/>
-  <limit upper="0.015" lower="0.0" effort="100" velocity="100"/>
-</joint>
-<joint name="jaw2" type="prismatic">
-  <origin xyz="0.007741 -0.039998 -0.030449" rpy="0 0 0"/>
-  <parent link="Gripper_1"/>
-  <child link="Right_jaw_1"/>
-  <axis xyz="0.0 -0.0 1.0"/>
-  <limit upper="0.015" lower="0.0" effort="100" velocity="100"/>
+  <limit lower="-3.14159265359" upper="3.14159265359" effort="100" velocity="2.0"/>
 </joint>
 </robot>
